File: NightLight.kicad_pcb (KiCad board)
At the start: 2 copper layers, 40 x 40 mm, 33 parts, among them Q1 BC817, Q2 BC817, U1 ESP32-C3-MINI-1, U2 LIS2DW12, U3 CP2102N, U4 LM1117-3.3, X1 USB_B_Micro, X2 Conn_01x04_Female

Commit message: Minor improvents and cleanups.
Parts:
- PB1: value SW_Push -> RESET
- moved R10 2.33 mm to (152.8, 86.8)
- moved R9 1.97 mm to (152.8, 91.6)
- moved R11 1.97 mm to (152.8, 89.2)
- moved D2 1.39 mm to (152.8, 81.8)
- moved D3 1.39 mm to (152.8, 84.3)
- moved R12 1.39 mm to (146.9, 84.3)
- moved R3 1.39 mm to (146.9, 81.8)
- moved X2 0.22 mm to (130.6, 113.2)
- moved R8 0.20 mm to (158.6, 91.2)
- moved C3 0.20 mm to (121.6, 82.8)
- moved C4 0.20 mm to (123.9, 82.8)
- moved X1 0.15 mm to (158.6, 100.0)
- moved U1 0.10 mm to (132.1, 86.0)
Connections:
- U1 pad 11: unconnected-(U1-Pad11) -> GND
- U1 pad 14: unconnected-(U1-Pad14) -> GND
- U1 pad 2: unconnected-(U1-Pad2) -> GND
- U1 pad 36: unconnected-(U1-Pad36) -> GND
- U1 pad 37: unconnected-(U1-Pad37) -> GND
- U1 pad 38: unconnected-(U1-Pad38) -> GND
- U1 pad 39: unconnected-(U1-Pad39) -> GND
- U1 pad 40: unconnected-(U1-Pad40) -> GND
- U1 pad 41: unconnected-(U1-Pad41) -> GND
- U1 pad 42: unconnected-(U1-Pad42) -> GND
- U1 pad 43: unconnected-(U1-Pad43) -> GND
- U1 pad 44: unconnected-(U1-Pad44) -> GND
- U1 pad 45: unconnected-(U1-Pad45) -> GND
- U1 pad 46: unconnected-(U1-Pad46) -> GND
- U1 pad 49: unconnected-(U1-Pad49) -> GND
- U1 pad 50: unconnected-(U1-Pad50) -> GND
- U1 pad 51: unconnected-(U1-Pad51) -> GND
- U1 pad 52: unconnected-(U1-Pad52) -> GND
- U1 pad 53: unconnected-(U1-Pad53) -> GND
Routing:
- net GND: track 52.6 -> 79.4 mm, vias 15 -> 25
- net /INT2: track 0.00 -> 14.7 mm, vias 0 -> 2
- net +3V3: track 150.8 -> 138.5 mm
- net /RESET: track 40.1 -> 35.4 mm
- net Net-(R10-Pad2): track 4.23 -> 6.65 mm
- net /INT1: track 15.5 -> 13.7 mm
- net Net-(R12-Pad1): track 8.94 -> 7.85 mm
- net Net-(R11-Pad1): track 7.03 -> 5.98 mm
- net /LEDC: track 24.7 -> 24.4 mm, vias 0 -> 1
- net /LEDD: track 24.2 -> 23.9 mm, vias 0 -> 1
- net VBUS: track 66.6 -> 66.8 mm, vias 1 -> 0
Other:
- outline, holes or cut-outs redrawn
- board text added: "Etnolit 2022"

Commit message: Final fixes. Ready for fab?
Parts:
- added G***: oshw_silkscreen-front_5mm, Etnolit:oshw_silkscreen-front_5mm, F.Cu at (124.0, 109.5)
- X1: footprint Custom:Wurth 629105136821 -> Etnolit:USB_B_Micro
- moved X1 1.74 mm to (156.9, 100.0)
Routing:
- net GND: track 79.4 -> 88.2 mm, vias 25 -> 24
Other:
- board text added: "NightLight v1"
