File: NightLight.kicad_sch (KiCad schematic)
At the start: 31 parts, among them Q1 BC817, Q2 BC817, U1 ESP32-C3-MINI-1, U2 LIS2DW12, U3 CP2102N, U4 LM1117-3.3, X1 USB_B_Micro, X2 Conn_01x04_Female

Commit message: Preliminary component placement on PCB.
Parts:
- added D3: LED, Diode_SMD:D_0805_2012Metric_Pad1.15x1.40mm_HandSolder, symbol Device:LED
- added R12: 1K, Resistor_SMD:R_0805_2012Metric_Pad1.20x1.40mm_HandSolder, symbol Device:R
- C2: value 10uF -> 22uF; footprint Capacitor_SMD:C_0805_2012Metric_Pad1.18x1.45mm_HandSolder -> Capacitor_SMD:CP_Elec_4x5.4
- C3: footprint Capacitor_SMD:C_0805_2012Metric_Pad1.18x1.45mm_HandSolder -> Capacitor_SMD:C_0805_2012Metric
- renumbered D2 to D1, D1 to D2
Connections:
- net GND: now also D3.1 (K); no longer U1.11 (GND11), U1.14 (GND14), U1.2 (GND2), U1.36 (GND36), U1.37 (GND37), U1.38 (GND38), U1.39 (GND39), U1.40 (GND40), U1.41 (GND41), U1.42 (GND42), U1.43 (GND43), U1.44 (GND44), U1.45 (GND45), U1.46 (GND46), U1.49 (pad1), U1.50 (GND50), U1.51 (GND51), U1.52 (GND52), U1.53 (GND53), U1.54 (pad2), U1.55 (pad3), U1.56 (pad4), U1.57 (pad5), U1.58 (pad6), U1.59 (pad7), U1.60 (pad8)
- net LEDC: now also X2.2 (Pin_2); no longer X2.3 (Pin_3)
- net LEDD: now also X2.3 (Pin_3); no longer X2.2 (Pin_2)
- net at U3.11 (~{SUSPEND}): now also R12.1
- new net: D3.2 (A), R12.2
- no-connect marks 25 -> 24
Other:
- moved on the sheet: C1, C2, D2, R3, U4

Commit message: Improved layout.
Parts:
- C3: footprint Capacitor_SMD:C_0805_2012Metric -> Capacitor_SMD:C_0805_2012Metric_Pad1.18x1.45mm_HandSolder
- D2: value LED -> PWR
- D3: value LED -> USB
Connections:
- net VBUS: now also D1.5 (K), R9.1, X1.1 (VBUS)
- net at U3.4 (D+), X1.2 (D-): now also D1.3 (K); no longer D1.1 (K)
- net at U3.5 (D-), X1.3 (D+): now also D1.1 (K); no longer D1.5 (K)
- net INT2: no longer names the net of U1.13 (IO1)
- net INT2: no longer U2.11 (INT2)
- now unconnected: D1.4 (K)
- no-connect marks 24 -> 26
Changed lines of the file:
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@@
   (junction (at 71.12 36.83) (diameter 0) (color 0 0 0 0)
   )
+  (junction (at 215.9 39.37) (diameter 0) (color 0 0 0 0)
+  )
+  (junction (at 35.56 36.83) (diameter 0) (color 0 0 0 0)
+  )
+  (junction (at 146.05 27.94) (diameter 0) (color 0 0 0 0)
+  )
+  (junction (at 146.05 63.5) (diameter 0) (color 0 0 0 0)
+  )
   (junction (at 215.9 68.58) (diameter 0) (color 0 0 0 0)
   )
-  (junction (at 35.56 36.83) (diameter 0) (color 0 0 0 0)
-  )
-  (junction (at 210.82 76.2) (diameter 0) (color 0 0 0 0)
-  )
-  (junction (at 146.05 27.94) (diameter 0) (color 0 0 0 0)
-  )
-  (junction (at 146.05 63.5) (diameter 0) (color 0 0 0 0)
-  )
   (junction (at 219.71 52.07) (diameter 0) (color 0 0 0 0)
   )
@@
   (junction (at 119.38 118.11) (diameter 0) (color 0 0 0 0)
   )
+  (junction (at 210.82 73.66) (diameter 0) (color 0 0 0 0)
+  )
   (junction (at 246.38 50.8) (diameter 0) (color 0 0 0 0)
   )
@@
   (junction (at 29.21 137.16) (diameter 0) (color 0 0 0 0)
   )
-  (junction (at 218.44 73.66) (diameter 0) (color 0 0 0 0)
-  )
   (junction (at 143.51 63.5) (diameter 0) (color 0 0 0 0)
   )
+  (junction (at 213.36 76.2) (diameter 0) (color 0 0 0 0)
+  )
   (junction (at 254 33.02) (diameter 0) (color 0 0 0 0)
   )
   (junction (at 177.8 124.46) (diameter 0) (color 0 0 0 0)
   )
-  (no_connect (at 213.36 82.55))
+  (no_connect (at 88.9 135.89))
+  (no_connect (at 215.9 80.01))
   (no_connect (at 88.9 153.67))
   (no_connect (at 57.15 139.7))
+  (no_connect (at 160.02 48.26))
   (no_connect (at 132.08 48.26))
   (no_connect (at 88.9 140.97))
@@
     (stroke (width 0) (type default) (color 0 0 0 0))
   )
+  (wire (pts (xy 210.82 73.66) (xy 210.82 83.82))
+    (stroke (width 0) (type default) (color 0 0 0 0))
+  )
   (wire (pts (xy 92.71 101.6) (xy 92.71 97.79))
     (stroke (width 0) (type default) (color 0 0 0 0))
@@
     (stroke (width 0) (type default) (color 0 0 0 0))
   )
-  (wire (pts (xy 218.44 73.66) (xy 218.44 83.82))
+  (wire (pts (xy 213.36 76.2) (xy 213.36 83.82))
     (stroke (width 0) (type default) (color 0 0 0 0))
   )
@@
     (stroke (width 0) (type default) (color 0 0 0 0))
   )
-  (wire (pts (xy 210.82 76.2) (xy 233.68 76.2))
+  (wire (pts (xy 205.74 76.2) (xy 213.36 76.2))
     (stroke (width 0) (type default) (color 0 0 0 0))
   )
@@
     (stroke (width 0) (type default) (color 0 0 0 0))
   )
+  (wire (pts (xy 218.44 83.82) (xy 218.44 68.58))
+    (stroke (width 0) (type default) (color 0 0 0 0))
+  )
   (wire (pts (xy 195.58 83.82) (xy 195.58 91.44))
     (stroke (width 0) (type default) (color 0 0 0 0))
@@
     (stroke (width 0) (type default) (color 0 0 0 0))
   )
-  (wire (pts (xy 218.44 73.66) (xy 233.68 73.66))
+  (wire (pts (xy 218.44 68.58) (xy 215.9 68.58))
     (stroke (width 0) (type default) (color 0 0 0 0))
   )
@@
     (stroke (width 0) (type default) (color 0 0 0 0))
   )
+  (wire (pts (xy 210.82 73.66) (xy 233.68 73.66))
+    (stroke (width 0) (type default) (color 0 0 0 0))
+  )
   (wire (pts (xy 35.56 33.02) (xy 35.56 36.83))
     (stroke (width 0) (type default) (color 0 0 0 0))
@@
     (stroke (width 0) (type default) (color 0 0 0 0))
   )
-  (wire (pts (xy 210.82 76.2) (xy 210.82 83.82))
-    (stroke (width 0) (type default) (color 0 0 0 0))
-  )
   (wire (pts (xy 260.35 104.14) (xy 259.08 104.14))
     (stroke (width 0) (type default) (color 0 0 0 0))
@@
     (stroke (width 0) (type default) (color 0 0 0 0))
   )
-  (wire (pts (xy 87.63 135.89) (xy 91.44 135.89))
-    (stroke (width 0) (type default) (color 0 0 0 0))
-  )
   (wire (pts (xy 29.21 142.24) (xy 29.21 137.16))
     (stroke (width 0) (type default) (color 0 0 0 0))
@@
     (stroke (width 0) (type default) (color 0 0 0 0))
   )
-  (wire (pts (xy 213.36 82.55) (xy 213.36 83.82))
+  (wire (pts (xy 215.9 80.01) (xy 215.9 83.82))
     (stroke (width 0) (type default) (color 0 0 0 0))
   )
@@
     (stroke (width 0) (type default) (color 0 0 0 0))
   )
+  (wire (pts (xy 215.9 36.83) (xy 215.9 39.37))
+    (stroke (width 0) (type default) (color 0 0 0 0))
+  )
   (wire (pts (xy 104.14 38.1) (xy 104.14 40.64))
     (stroke (width 0) (type default) (color 0 0 0 0))
@@
     (stroke (width 0) (type default) (color 0 0 0 0))
   )
+  (wire (pts (xy 205.74 73.66) (xy 210.82 73.66))
+    (stroke (width 0) (type default) (color 0 0 0 0))
+  )
   (wire (pts (xy 49.53 142.24) (xy 58.42 142.24))
     (stroke (width 0) (type default) (color 0 0 0 0))
@@
     (stroke (width 0) (type default) (color 0 0 0 0))
   )
-  (wire (pts (xy 215.9 68.58) (xy 215.9 83.82))
+  (wire (pts (xy 213.36 76.2) (xy 233.68 76.2))
     (stroke (width 0) (type default) (color 0 0 0 0))
   )
@@
     (stroke (width 0) (type default) (color 0 0 0 0))
   )
+  (wire (pts (xy 87.63 135.89) (xy 88.9 135.89))
+    (stroke (width 0) (type default) (color 0 0 0 0))
+  )
   (wire (pts (xy 92.71 97.79) (xy 87.63 97.79))
     (stroke (width 0) (type default) (color 0 0 0 0))
@@
     (stroke (width 0) (type default) (color 0 0 0 0))
   )
-  (wire (pts (xy 205.74 76.2) (xy 210.82 76.2))
-    (stroke (width 0) (type default) (color 0 0 0 0))
-  )
   (wire (pts (xy 207.01 78.74) (xy 205.74 78.74))
     (stroke (width 0) (type default) (color 0 0 0 0))
@@
   )
   (wire (pts (xy 260.35 68.58) (xy 259.08 68.58))
-    (stroke (width 0) (type default) (color 0 0 0 0))
-  )
-  (wire (pts (xy 205.74 73.66) (xy 218.44 73.66))
     (stroke (width 0) (type default) (color 0 0 0 0))
   )
@@
   )
   (label "SDA" (at 125.73 45.72 0)
-    (effects (font (size 1.27 1.27)) (justify left bottom))
-  )
-  (label "INT2" (at 160.02 48.26 0)
-    (effects (font (size 1.27 1.27)) (justify left bottom))
-  )
-  (label "INT2" (at 91.44 135.89 0)
     (effects (font (size 1.27 1.27)) (justify left bottom))
   )
@@
       (effects (font (size 1.27 1.27)) (justify left))
     )
-    (property "Footprint" "Capacitor_SMD:C_0805_2012Metric" (id 2) (at 30.1752 149.86 0)
+    (property "Footprint" "Capacitor_SMD:C_0805_2012Metric_Pad1.18x1.45mm_HandSolder" (id 2) (at 30.1752 149.86 0)
       (effects (font (size 1.27 1.27)) hide)
     )
@@
       (effects (font (size 1.27 1.27)) (justify right))
     )
-    (property "Value" "LED" (id 1) (at 107.95 47.3074 90)
+    (property "Value" "PWR" (id 1) (at 107.95 47.3074 90)
       (effects (font (size 1.27 1.27)) (justify right))
     )
@@
     )
     (property "Datasheet" "" (id 3) (at 182.88 40.64 0)
+      (effects (font (size 1.27 1.27)) hide)
+    )
+    (pin "1")
+  )
+  (symbol (lib_id "power:VBUS") (at 215.9 36.83 0) (unit 1)
+    (in_bom yes) (on_board yes) (fields_autoplaced)
+    (property "Reference" "#PWR0105" (id 0) (at 215.9 40.64 0)
+      (effects (font (size 1.27 1.27)) hide)
+    )
+    (property "Value" "VBUS" (id 1) (at 215.9 31.75 0))
+    (property "Footprint" "" (id 2) (at 215.9 36.83 0)
+      (effects (font (size 1.27 1.27)) hide)
+    )
+    (property "Datasheet" "" (id 3) (at 215.9 36.83 0)
       (effects (font (size 1.27 1.27)) hide)
     )
@@
       (effects (font (size 1.27 1.27)) (justify right))
     )
-    (property "Value" "LED" (id 1) (at 275.59 103.1874 90)
+    (property "Value" "USB" (id 1) (at 275.59 103.1874 90)
       (effects (font (size 1.27 1.27)) (justify right))
     )
@@
       (reference "#PWR0104") (unit 1) (value "GND") (footprint "")
     )
+    (path "/c0ed410a-0280-4a8c-8ff3-f58b7b1340fc"
+      (reference "#PWR0105") (unit 1) (value "VBUS") (footprint "")
+    )
     (path "/0feaa0e3-c0f0-4d3c-8a22-243f972f44bf"
       (reference "C1") (unit 1) (value "10uF") (footprint "Capacitor_SMD:C_0805_2012Metric_Pad1.18x1.45mm_HandSolder")
@@
     )
     (path "/3cdff4de-163a-4433-88b6-dddbb131d19a"
-      (reference "C3") (unit 1) (value "10uF") (footprint "Capacitor_SMD:C_0805_2012Metric")
+      (reference "C3") (unit 1) (value "10uF") (footprint "Capacitor_SMD:C_0805_2012Metric_Pad1.18x1.45mm_HandSolder")
     )
     (path "/e07b1e88-c521-4e06-9394-f1a3ff44357c"
@@
     )
     (path "/b7b373c7-819c-4980-8b57-6917235d1dc7"
-      (reference "D2") (unit 1) (value "LED") (footprint "Diode_SMD:D_0805_2012Metric_Pad1.15x1.40mm_HandSolder")
+      (reference "D2") (unit 1) (value "PWR") (footprint "Diode_SMD:D_0805_2012Metric_Pad1.15x1.40mm_HandSolder")
     )
     (path "/f2187aab-7d18-4338-8c36-b3c4d9fa94dd"
-      (reference "D3") (unit 1) (value "LED") (footprint "Diode_SMD:D_0805_2012Metric_Pad1.15x1.40mm_HandSolder")
+      (reference "D3") (unit 1) (value "USB") (footprint "Diode_SMD:D_0805_2012Metric_Pad1.15x1.40mm_HandSolder")
     )
     (path "/9358e013-3f01-4ec1-804d-cf8481494d82"

Commit message: WIP
Changed lines of the file:
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@@
     (pin "47")
     (pin "48")
-    (pin "49")
     (pin "50")
     (pin "51")
     (pin "52")
     (pin "53")
-    (pin "54")
-    (pin "55")
-    (pin "56")
-    (pin "57")
-    (pin "58")
-    (pin "59")
-    (pin "60")
     (pin "1")
     (pin "10")

Commit message: Minor improvents and cleanups.
Parts:
- PB1: value SW_Push -> RESET
Connections:
- net GND: now also U1.11 (GND11), U1.14 (GND14), U1.2 (GND2), U1.36 (GND36), U1.37 (GND37), U1.38 (GND38), U1.39 (GND39), U1.40 (GND40), U1.41 (GND41), U1.42 (GND42), U1.43 (GND43), U1.44 (GND44), U1.45 (GND45), U1.46 (GND46), U1.49 (GND_PAD), U1.50 (GND50), U1.51 (GND51), U1.52 (GND52), U1.53 (GND53)
- net INT2: now reaches U1.13 (IO1)
- net INT2: now also U2.11 (INT2)
- no-connect marks 26 -> 24

Commit message: Final fixes. Ready for fab?
Parts:
- U1: symbol esp32-c3-mini-1:ESP32-C3-MINI-1 -> Etnolit:ESP32-C3-MINI-1
- X1: footprint Connector_USB:USB_Micro-B_Wuerth_629105150521 -> Etnolit:USB_B_Micro
Other:
- moved on the sheet: C3, C4, R1, R2
